Commit message: feat(robot_mima_mkv30): [2405-01] add simulation plugin defaults
Add the staged bridge and simulation example configuration for the MiMA MKV30 models and include the shared Gazebo system plugin macros from common.xacro. This makes the model examples carry the simulation plugin setup needed by downstream launch stacks.

File: urdf/includes/common.xacro (robot description, xacro)
@@ -3,4 +3,5 @@
   <xacro:include filename="$(find robotics_description)/urdf/common/all_commons.xacro"/>
   <xacro:include filename="$(find robotics_description)/urdf/wheels/all_wheels.xacro"/>
+  <xacro:include filename="$(find robotics_description)/urdf/gz_system_plugins/all_gz_system_plugins.xacro"/>
   <xacro:include filename="$(find robot_mima_mkv30)/urdf/includes/fork_macro.xacro"/>
   <xacro:arg name="use_sim_mode" default="False"/>
@@ -70,5 +71,5 @@
   <!-- Steerable wheel launch-facing properties. -->
   <xacro:property name="s_wheel_use_v_mesh"              value="$(arg s_wheel_use_v_mesh)"/>
-  <xacro:property name="s_wheel_color"                   value="0 1 0 1"/>
+  <xacro:property name="s_wheel_color"                   value="0 0 0 1"/>
   <xacro:property name="s_wheel_steering_joint_limits"   value="$(arg s_wheel_steering_joint_limits)"/>
   <xacro:property name="s_wheel_steering_joint_dynamics" value="$(arg s_wheel_steering_joint_dynamics)"/>
@@ -95,5 +96,5 @@
   <xacro:property name="wheel_use_inertial"              value="$(arg wheel_use_inertial)"/>
   <xacro:property name="wheel_use_v_mesh"                value="$(arg wheel_use_v_mesh)"/>
-  <xacro:property name="wheel_color"                     value="0 1 0 1"/>
+  <xacro:property name="wheel_color"                     value="0 0 0 1"/>
   <xacro:property name="wheel_rotation_joint_limits"     value="$(arg wheel_rotation_joint_limits)"/>
   <xacro:property name="wheel_rotation_joint_dynamics"   value="$(arg wheel_rotation_joint_dynamics)"/>
@@ -148,4 +149,53 @@
     <origin rpy="0 0 0" xyz="0 0 ${wheel_radius}"/>
   </joint>
+  <xacro:property name="base_pose_ground_truth_publisher_sim_cfg"
+                  value="${sim_cfg.get('base_pose_ground_truth_publisher', dict())}"/>
+  <xacro:if value="${base_pose_ground_truth_publisher_sim_cfg.get('enabled', False)}">
+    <!--
+    Prepend the prefix `bpgtp_` to all properties related to the base pose ground
+    truth publisher Gazebo plugin, to avoid name conflicts with other Gazebo plugins.
+    -->
+    <xacro:property name="bpgtp_nav_topic_no_cov"
+                    value="${base_pose_ground_truth_publisher_sim_cfg.get('nav_topic_no_cov', '')}"/>
+    <xacro:property name="bpgtp_nav_topic_cov"
+                    value="${base_pose_ground_truth_publisher_sim_cfg.get('nav_topic_cov', '')}"/>
+    <xacro:property name="bpgtp_tf_topic"
+                    value="${base_pose_ground_truth_publisher_sim_cfg.get('tf_topic', '')}"/>
+    <!-- If one of the topics is empty, then the plugin is not loaded. -->
+    <xacro:if value="${bpgtp_nav_topic_cov != '' and bpgtp_nav_topic_no_cov != '' and bpgtp_tf_topic != ''}">
+      <xacro:resolve_topic prop_id="bpgtp_resolved_nav_topic_cov"
+                           topic="${bpgtp_nav_topic_cov}"
+                           namespace="${robot_namespace}"/>
+      <xacro:resolve_topic prop_id="bpgtp_resolved_nav_topic_no_cov"
+                           topic="${bpgtp_nav_topic_no_cov}"
+                           namespace="${robot_namespace}"/>
+      <xacro:resolve_topic prop_id="bpgtp_resolved_tf_topic"
+                           topic="${bpgtp_tf_topic}"
+                           namespace="${robot_namespace}"/>
+      <xacro:property name="bpgtp_fixed_frame"
+                      value="${base_pose_ground_truth_publisher_sim_cfg.get('fixed_frame', 'sim_world')}"/>
+      <xacro:property name="bpgtp_offset"
+                      value="${base_pose_ground_truth_publisher_sim_cfg.get('offset', dict(x=0, y=0, z=0, R=0, P=0, Y=0))}"/>
+      <xacro:property name="bpgtp_global_offset"
+                      value="${base_pose_ground_truth_publisher_sim_cfg.get('global_offset', dict(x=0, y=0, z=0, R=0, P=0, Y=0))}"/>
+      <xacro:property name="bpgtp_gaussian_noise"
+                      value="${base_pose_ground_truth_publisher_sim_cfg.get('gaussian_noise', 0)}"/>
+      <xacro:property name="bpgtp_publication_frequency"
+                      value="${base_pose_ground_truth_publisher_sim_cfg.get('publication_frequency', 50)}"/>
+      <xacro:plugin_odometry_publisher
+        odom_frame="${bpgtp_fixed_frame}"
+        robot_base_frame="${robot_prefix}base_footprint_link"
+        odom_publish_frequency="${bpgtp_publication_frequency}"
+        odom_topic="${bpgtp_resolved_nav_topic_no_cov}"
+        odom_covariance_topic="${bpgtp_resolved_nav_topic_cov}"
+        tf_topic="${bpgtp_resolved_tf_topic}"
+        dimensions="2"
+        xyz_offset="${bpgtp_offset['x']} ${bpgtp_offset['y']} ${bpgtp_offset['z']}"
+        rpy_offset="${bpgtp_offset['R']} ${bpgtp_offset['P']} ${bpgtp_offset['Y']}"
+        xyz_global_offset="${bpgtp_global_offset['x']} ${bpgtp_global_offset['y']} ${bpgtp_global_offset['z']}"
+        rpy_global_offset="${bpgtp_global_offset['R']} ${bpgtp_global_offset['P']} ${bpgtp_global_offset['Y']}"
+        gaussian_noise="${bpgtp_gaussian_noise}"/>
+    </xacro:if>
+  </xacro:if>
   <link name="${robot_prefix}chassis_link">
     <xacro:if value="${chassis_use_visual}">

Commit message: fix(xacro): [2605-02] keep shared sim defaults explicit
Leave shared xacro arguments empty so model-specific controller and simulation files come from the xargs contract instead of common.xacro defaults. Keep the xargs sync test focused on defaults that are common across models.

File: urdf/includes/common.xacro (robot description, xacro)
@@ -9,6 +9,5 @@
   <xacro:arg name="namespace"    default=""/>
   <xacro:arg name="robot_name"   default="mima_mkv30"/>
-  <xacro:arg name="controller_config_file"
-             default="$(find robot_mima_mkv30)/config/model_base/example_controllers.yaml.in"/>
+  <xacro:arg name="controller_config_file" default=""/>
   <!-- Chassis arguments. -->
   <xacro:arg name="chassis_use_visual"    default="True"/>
@@ -149,53 +148,4 @@
     <origin rpy="0 0 0" xyz="0 0 ${wheel_radius}"/>
   </joint>
-  <xacro:property name="base_pose_ground_truth_publisher_sim_cfg"
-                  value="${sim_cfg.get('base_pose_ground_truth_publisher', dict())}"/>
-  <xacro:if value="${base_pose_ground_truth_publisher_sim_cfg.get('enabled', False)}">
-    <!--
-    Prepend the prefix `bpgtp_` to all properties related to the base pose ground
-    truth publisher Gazebo plugin, to avoid name conflicts with other Gazebo plugins.
-    -->
-    <xacro:property name="bpgtp_nav_topic_no_cov"
-                    value="${base_pose_ground_truth_publisher_sim_cfg.get('nav_topic_no_cov', '')}"/>
-    <xacro:property name="bpgtp_nav_topic_cov"
-                    value="${base_pose_ground_truth_publisher_sim_cfg.get('nav_topic_cov', '')}"/>
-    <xacro:property name="bpgtp_tf_topic"
-                    value="${base_pose_ground_truth_publisher_sim_cfg.get('tf_topic', '')}"/>
-    <!-- If one of the topics is empty, then the plugin is not loaded. -->
-    <xacro:if value="${bpgtp_nav_topic_cov != '' and bpgtp_nav_topic_no_cov != '' and bpgtp_tf_topic != ''}">
-      <xacro:resolve_topic prop_id="bpgtp_resolved_nav_topic_cov"
-                           topic="${bpgtp_nav_topic_cov}"
-                           namespace="${robot_namespace}"/>
-      <xacro:resolve_topic prop_id="bpgtp_resolved_nav_topic_no_cov"
-                           topic="${bpgtp_nav_topic_no_cov}"
-                           namespace="${robot_namespace}"/>
-      <xacro:resolve_topic prop_id="bpgtp_resolved_tf_topic"
-                           topic="${bpgtp_tf_topic}"
-                           namespace="${robot_namespace}"/>
-      <xacro:property name="bpgtp_fixed_frame"
-                      value="${base_pose_ground_truth_publisher_sim_cfg.get('fixed_frame', 'sim_world')}"/>
-      <xacro:property name="bpgtp_offset"
-                      value="${base_pose_ground_truth_publisher_sim_cfg.get('offset', dict(x=0, y=0, z=0, R=0, P=0, Y=0))}"/>
-      <xacro:property name="bpgtp_global_offset"
-                      value="${base_pose_ground_truth_publisher_sim_cfg.get('global_offset', dict(x=0, y=0, z=0, R=0, P=0, Y=0))}"/>
-      <xacro:property name="bpgtp_gaussian_noise"
-                      value="${base_pose_ground_truth_publisher_sim_cfg.get('gaussian_noise', 0)}"/>
-      <xacro:property name="bpgtp_publication_frequency"
-                      value="${base_pose_ground_truth_publisher_sim_cfg.get('publication_frequency', 50)}"/>
-      <xacro:plugin_odometry_publisher
-        odom_frame="${bpgtp_fixed_frame}"
-        robot_base_frame="${robot_prefix}base_footprint_link"
-        odom_publish_frequency="${bpgtp_publication_frequency}"
-        odom_topic="${bpgtp_resolved_nav_topic_no_cov}"
-        odom_covariance_topic="${bpgtp_resolved_nav_topic_cov}"
-        tf_topic="${bpgtp_resolved_tf_topic}"
-        dimensions="2"
-        xyz_offset="${bpgtp_offset['x']} ${bpgtp_offset['y']} ${bpgtp_offset['z']}"
-        rpy_offset="${bpgtp_offset['R']} ${bpgtp_offset['P']} ${bpgtp_offset['Y']}"
-        xyz_global_offset="${bpgtp_global_offset['x']} ${bpgtp_global_offset['y']} ${bpgtp_global_offset['z']}"
-        rpy_global_offset="${bpgtp_global_offset['R']} ${bpgtp_global_offset['P']} ${bpgtp_global_offset['Y']}"
-        gaussian_noise="${bpgtp_gaussian_noise}"/>
-    </xacro:if>
-  </xacro:if>
   <link name="${robot_prefix}chassis_link">
     <xacro:if value="${chassis_use_visual}">
@@ -361,3 +311,63 @@
               y_left_tine="${fork_y_left_tine}"
               y_right_tine="${fork_y_right_tine}"/>
+  <xacro:if value="${use_sim_mode}">
+    <gazebo>
+      <!--
+      Insert the `OdometryPublisher` Gazebo plugin to publish the true pose of
+      the robot with respect to a selected fixed frame in Gazebo.
+      More details about this plugin in
+      package://robotics_description/urdf/gz_system_plugins/plugin_odometry_publisher_macro.xacro
+      -->
+      <xacro:property name="base_pose_ground_truth_publisher_sim_cfg"
+                      value="${sim_cfg.get('base_pose_ground_truth_publisher', dict())}"/>
+      <xacro:if value="${base_pose_ground_truth_publisher_sim_cfg.get('enabled', False)}">
+        <!--
+        Prepend the prefix `bpgtp_` to all properties related to the base pose
+        ground truth publisher Gazebo plugin, to avoid name conflicts with
+        other Gazebo plugins.
+        -->
+        <xacro:property name="bpgtp_nav_topic_no_cov"
+                        value="${base_pose_ground_truth_publisher_sim_cfg.get('nav_topic_no_cov', '')}"/>
+        <xacro:property name="bpgtp_nav_topic_cov"
+                        value="${base_pose_ground_truth_publisher_sim_cfg.get('nav_topic_cov', '')}"/>
+        <xacro:property name="bpgtp_tf_topic"
+                        value="${base_pose_ground_truth_publisher_sim_cfg.get('tf_topic', '')}"/>
+        <!-- If one of the topics is empty, then the plugin is not loaded. -->
+        <xacro:if value="${bpgtp_nav_topic_cov != '' and bpgtp_nav_topic_no_cov != '' and bpgtp_tf_topic != ''}">
+          <xacro:resolve_topic prop_id="bpgtp_resolved_nav_topic_cov"
+                               topic="${bpgtp_nav_topic_cov}"
+                               namespace="${robot_namespace}"/>
+          <xacro:resolve_topic prop_id="bpgtp_resolved_nav_topic_no_cov"
+                               topic="${bpgtp_nav_topic_no_cov}"
+                               namespace="${robot_namespace}"/>
+          <xacro:resolve_topic prop_id="bpgtp_resolved_tf_topic"
+                               topic="${bpgtp_tf_topic}"
+                               namespace="${robot_namespace}"/>
+          <xacro:property name="bpgtp_fixed_frame"
+                          value="${base_pose_ground_truth_publisher_sim_cfg.get('fixed_frame', 'sim_world')}"/>
+          <xacro:property name="bpgtp_offset"
+                          value="${base_pose_ground_truth_publisher_sim_cfg.get('offset', dict(x=0, y=0, z=0, R=0, P=0, Y=0))}"/>
+          <xacro:property name="bpgtp_global_offset"
+                          value="${base_pose_ground_truth_publisher_sim_cfg.get('global_offset', dict(x=0, y=0, z=0, R=0, P=0, Y=0))}"/>
+          <xacro:property name="bpgtp_gaussian_noise"
+                          value="${base_pose_ground_truth_publisher_sim_cfg.get('gaussian_noise', 0)}"/>
+          <xacro:property name="bpgtp_publication_frequency"
+                          value="${base_pose_ground_truth_publisher_sim_cfg.get('publication_frequency', 50)}"/>
+          <xacro:plugin_odometry_publisher
+            odom_frame="${bpgtp_fixed_frame}"
+            robot_base_frame="${robot_prefix}base_footprint_link"
+            odom_publish_frequency="${bpgtp_publication_frequency}"
+            odom_topic="${bpgtp_resolved_nav_topic_no_cov}"
+            odom_covariance_topic="${bpgtp_resolved_nav_topic_cov}"
+            tf_topic="${bpgtp_resolved_tf_topic}"
+            dimensions="2"
+            xyz_offset="${bpgtp_offset['x']} ${bpgtp_offset['y']} ${bpgtp_offset['z']}"
+            rpy_offset="${bpgtp_offset['R']} ${bpgtp_offset['P']} ${bpgtp_offset['Y']}"
+            xyz_global_offset="${bpgtp_global_offset['x']} ${bpgtp_global_offset['y']} ${bpgtp_global_offset['z']}"
+            rpy_global_offset="${bpgtp_global_offset['R']} ${bpgtp_global_offset['P']} ${bpgtp_global_offset['Y']}"
+            gaussian_noise="${bpgtp_gaussian_noise}"/>
+        </xacro:if>
+      </xacro:if>
+    </gazebo>
+  </xacro:if>
 </robot>

Commit message: refactor(robot_mima_mkv30): [2905-01] consolidate robot parameter launch config
Unify robot parameter files for RSP, bridge, and ros2_control, update launch handling for rendered parameter files, and pin robotics_description to the commit that documents odometry publisher frame semantics.

File: urdf/includes/common.xacro (robot description, xacro)
@@ -5,9 +5,9 @@
   <xacro:include filename="$(find robotics_description)/urdf/gz_system_plugins/all_gz_system_plugins.xacro"/>
   <xacro:include filename="$(find robot_mima_mkv30)/urdf/includes/fork_macro.xacro"/>
-  <xacro:arg name="use_sim_mode" default="False"/>
-  <xacro:arg name="sim_file"     default=""/>
-  <xacro:arg name="namespace"    default=""/>
-  <xacro:arg name="robot_name"   default="mima_mkv30"/>
-  <xacro:arg name="controller_config_file" default=""/>
+  <xacro:arg name="use_sim_mode"           default="False"/>
+  <xacro:arg name="sim_file"               default=""/>
+  <xacro:arg name="namespace"              default=""/>
+  <xacro:arg name="robot_name"             default="mima_mkv30"/>
+  <xacro:arg name="ros2_control_config_file" default=""/>
   <!-- Chassis arguments. -->
   <xacro:arg name="chassis_use_visual"    default="True"/>
@@ -61,5 +61,5 @@
   <xacro:property name="rear_wheel_track"         value="1.1"/>
   <!-- Chassis fixed model properties. -->
-  <xacro:property name="chassis_color"           value="0 0 0.8 1.0"/>
+  <xacro:property name="chassis_color"           value="0.831372549 0 0 1"/>
   <xacro:property name="chassis_use_visual"      value="$(arg chassis_use_visual)"/>
   <xacro:property name="chassis_use_inertial"    value="$(arg chassis_use_inertial)"/>
@@ -115,7 +115,7 @@
   <xacro:property name="wheel_mass"                      value="100.0"/>
   <!-- Fork launch-facing properties. -->
-  <xacro:property name="fork_mast_color"        value="1 0 0 1"/>
-  <xacro:property name="fork_board_color"       value="0 0 1 1"/>
-  <xacro:property name="fork_tine_color"        value="0 1 0 1"/>
+  <xacro:property name="fork_mast_color"        value="0.2 0.2 0.2 1"/>
+  <xacro:property name="fork_board_color"       value="0.4 0.4 0.4 1"/>
+  <xacro:property name="fork_tine_color"        value="0.6 0.6 0.6 1"/>
   <xacro:property name="fork_use_visual"        value="$(arg fork_use_visual)"/>
   <xacro:property name="fork_use_inertial"      value="$(arg fork_use_inertial)"/>

File: urdf/includes/ros2_control_real_macro.xacro (robot description, xacro)
@@ -1,5 +1,5 @@
 <?xml version="1.0"?>
 <robot name="mima_mkv30_ros2_control_real_macro" xmlns:xacro="http://www.ros.org/wiki/xacro">
-  <xacro:macro name="mima_mkv30_ros2_control_real" params="controller_config_file">
+  <xacro:macro name="mima_mkv30_ros2_control_real" params="ros2_control_config_file">
     <!--
     Placeholder for real ros2_control integration.

File: urdf/includes/ros2_control_sim_macro.xacro (robot description, xacro)
@@ -1,5 +1,5 @@
 <?xml version="1.0"?>
 <robot name="ros2_control_sim_macro" xmlns:xacro="http://www.ros.org/wiki/xacro">
-  <xacro:macro name="ros2_control_sim" params="controller_config_file robot_namespace">
+  <xacro:macro name="ros2_control_sim" params="ros2_control_config_file robot_namespace">
     <ros2_control name="GazeboSimSystem" type="system">
       <hardware>
@@ -83,5 +83,5 @@
           <namespace>${robot_namespace}</namespace>
         </ros>
-        <parameters>${controller_config_file}</parameters>
+        <parameters>${ros2_control_config_file}</parameters>
       </plugin>
     </gazebo>

File: urdf/models/model_base.xacro (robot description, xacro)
@@ -11,5 +11,5 @@
   <xacro:if value="${use_sim_mode}">
     <xacro:ros2_control_sim
-      controller_config_file="$(arg controller_config_file)"
+      ros2_control_config_file="$(arg ros2_control_config_file)"
       robot_namespace="${robot_namespace}"/>
   </xacro:if>

File: urdf/models/model_sensors1.xacro (robot description, xacro)
@@ -498,5 +498,5 @@
   <xacro:if value="${use_sim_mode}">
     <xacro:ros2_control_sim
-      controller_config_file="$(arg controller_config_file)"
+      ros2_control_config_file="$(arg ros2_control_config_file)"
       robot_namespace="${robot_namespace}"/>
   </xacro:if>

Commit message: fix(urdf): [2905-02] align fork visuals and wheel friction frame
Update fork visual colors and use the base footprint frame for wheel friction direction references in the common robot xacro.

File: urdf/includes/common.xacro (robot description, xacro)
@@ -116,6 +116,6 @@
   <!-- Fork launch-facing properties. -->
   <xacro:property name="fork_mast_color"        value="0.2 0.2 0.2 1"/>
-  <xacro:property name="fork_board_color"       value="0.4 0.4 0.4 1"/>
-  <xacro:property name="fork_tine_color"        value="0.6 0.6 0.6 1"/>
+  <xacro:property name="fork_board_color"       value="0.8 0.8 0.8 1"/>
+  <xacro:property name="fork_tine_color"        value="0.95 0.95 0.95 1"/>
   <xacro:property name="fork_use_visual"        value="$(arg fork_use_visual)"/>
   <xacro:property name="fork_use_inertial"      value="$(arg fork_use_inertial)"/>
@@ -263,5 +263,5 @@
     sim_slip2="${rear_left_wheel_sim_slip2}"
     sim_fdir1="1 0 0"
-    sim_fdir1_frame="${robot_prefix}base_link"/>
+    sim_fdir1_frame="${robot_prefix}base_footprint_link"/>
   <xacro:property name="rear_right_wheel_sim_cfg"
                   value="${sim_cfg.get('rear_right_wheel', dict())}"/>
@@ -291,5 +291,5 @@
     sim_slip2="${rear_right_wheel_sim_slip2}"
     sim_fdir1="1 0 0"
-    sim_fdir1_frame="${robot_prefix}base_link"/>
+    sim_fdir1_frame="${robot_prefix}base_footprint_link"/>
   <xacro:fork prefix="${robot_prefix}"
               name="fork"
