Commit message: refactor(model-config)!: [1806-03] use model xacro args files
Replace the old properties-file contract with model_xacro_args_file YAML inputs passed to xacro as regular arguments. Update the model launch files, xacro models, example configuration files, and tests so model configuration is loaded through the new contract while launch-scoped values remain direct launch arguments.

File: urdf/models/model_sensors1.xacro (robot description, xacro)
@@ -8,66 +8,117 @@
   <xacro:include filename="$(find robot_mima_mkv30)/urdf/includes/ros2_control_sim_macro.xacro"/>
   <xacro:include filename="$(find robot_mima_mkv30)/urdf/includes/ros2_control_real_macro.xacro"/>
-  <!-- Model properties loaded from the file passed through the `properties_file` Xacro argument. -->
-  <xacro:property name="use_front_lidar2d"                           value="${properties_cfg.get('use_front_lidar2d', True)}"/>
-  <xacro:property name="front_lidar2d_use_visual"                    value="${properties_cfg.get('front_lidar2d_use_visual', True)}"/>
-  <xacro:property name="front_lidar2d_use_collision"                 value="${properties_cfg.get('front_lidar2d_use_collision', True)}"/>
-  <xacro:property name="front_lidar2d_use_v_mesh"                    value="${properties_cfg.get('front_lidar2d_use_v_mesh', True)}"/>
-  <xacro:property name="front_lidar2d_v_mesh_use_low_res"            value="${properties_cfg.get('front_lidar2d_v_mesh_use_low_res', True)}"/>
-  <xacro:property name="front_lidar2d_color"                         value="1 0.831372549 0.164705882 1"/>
-  <xacro:property name="front_lidar2d_use_c_mesh"                    value="${properties_cfg.get('front_lidar2d_use_c_mesh', False)}"/>
-  <xacro:property name="front_lidar2d_c_mesh_use_low_res"            value="${properties_cfg.get('front_lidar2d_c_mesh_use_low_res', True)}"/>
-  <xacro:property name="front_lidar2d_mount"                         value="2.1 0.0 -0.1 0 0 0"/>
-  <xacro:property name="use_back_lidar2d"                            value="${properties_cfg.get('use_back_lidar2d', True)}"/>
-  <xacro:property name="back_lidar2d_use_visual"                     value="${properties_cfg.get('back_lidar2d_use_visual', True)}"/>
-  <xacro:property name="back_lidar2d_use_collision"                  value="${properties_cfg.get('back_lidar2d_use_collision', True)}"/>
-  <xacro:property name="back_lidar2d_use_v_mesh"                     value="${properties_cfg.get('back_lidar2d_use_v_mesh', True)}"/>
-  <xacro:property name="back_lidar2d_v_mesh_use_low_res"             value="${properties_cfg.get('back_lidar2d_v_mesh_use_low_res', True)}"/>
-  <xacro:property name="back_lidar2d_color"                          value="1 0.831372549 0.164705882 1"/>
-  <xacro:property name="back_lidar2d_use_c_mesh"                     value="${properties_cfg.get('back_lidar2d_use_c_mesh', False)}"/>
-  <xacro:property name="back_lidar2d_c_mesh_use_low_res"             value="${properties_cfg.get('back_lidar2d_c_mesh_use_low_res', True)}"/>
-  <xacro:property name="back_lidar2d_mount"                          value="-0.7 0.0 -0.1 0 0 ${-pi}"/>
-  <xacro:property name="use_left_lidar2d"                            value="${properties_cfg.get('use_left_lidar2d', True)}"/>
-  <xacro:property name="left_lidar2d_use_visual"                     value="${properties_cfg.get('left_lidar2d_use_visual', True)}"/>
-  <xacro:property name="left_lidar2d_use_collision"                  value="${properties_cfg.get('left_lidar2d_use_collision', True)}"/>
-  <xacro:property name="left_lidar2d_use_v_mesh"                     value="${properties_cfg.get('left_lidar2d_use_v_mesh', True)}"/>
-  <xacro:property name="left_lidar2d_v_mesh_use_low_res"             value="${properties_cfg.get('left_lidar2d_v_mesh_use_low_res', True)}"/>
-  <xacro:property name="left_lidar2d_color"                          value="1 0.831372549 0.164705882 1"/>
-  <xacro:property name="left_lidar2d_use_c_mesh"                     value="${properties_cfg.get('left_lidar2d_use_c_mesh', False)}"/>
-  <xacro:property name="left_lidar2d_c_mesh_use_low_res"             value="${properties_cfg.get('left_lidar2d_c_mesh_use_low_res', True)}"/>
-  <xacro:property name="left_lidar2d_mount"                          value="0.4 0.7 -0.1 0 0 ${0.5 * pi}"/>
-  <xacro:property name="use_right_lidar2d"                           value="${properties_cfg.get('use_right_lidar2d', True)}"/>
-  <xacro:property name="right_lidar2d_use_visual"                    value="${properties_cfg.get('right_lidar2d_use_visual', True)}"/>
-  <xacro:property name="right_lidar2d_use_collision"                 value="${properties_cfg.get('right_lidar2d_use_collision', True)}"/>
-  <xacro:property name="right_lidar2d_use_v_mesh"                    value="${properties_cfg.get('right_lidar2d_use_v_mesh', True)}"/>
-  <xacro:property name="right_lidar2d_v_mesh_use_low_res"            value="${properties_cfg.get('right_lidar2d_v_mesh_use_low_res', True)}"/>
-  <xacro:property name="right_lidar2d_color"                         value="1 0.831372549 0.164705882 1"/>
-  <xacro:property name="right_lidar2d_use_c_mesh"                    value="${properties_cfg.get('right_lidar2d_use_c_mesh', False)}"/>
-  <xacro:property name="right_lidar2d_c_mesh_use_low_res"            value="${properties_cfg.get('right_lidar2d_c_mesh_use_low_res', True)}"/>
-  <xacro:property name="right_lidar2d_mount"                         value="1.4 -0.7 -0.1 0 0 ${-0.5 * pi}"/>
-  <xacro:property name="use_front_top_lidar3d"                       value="${properties_cfg.get('use_front_top_lidar3d', True)}"/>
-  <xacro:property name="front_top_lidar3d_use_visual"                value="${properties_cfg.get('front_top_lidar3d_use_visual', True)}"/>
-  <xacro:property name="front_top_lidar3d_use_collision"             value="${properties_cfg.get('front_top_lidar3d_use_collision', True)}"/>
-  <xacro:property name="front_top_lidar3d_use_v_mesh"                value="${properties_cfg.get('front_top_lidar3d_use_v_mesh', True)}"/>
-  <xacro:property name="front_top_lidar3d_v_mesh_use_low_res"        value="${properties_cfg.get('front_top_lidar3d_v_mesh_use_low_res', True)}"/>
-  <xacro:property name="front_top_lidar3d_color"                     value="0 0 0 1"/>
-  <xacro:property name="front_top_lidar3d_use_c_mesh"                value="${properties_cfg.get('front_top_lidar3d_use_c_mesh', False)}"/>
-  <xacro:property name="front_top_lidar3d_c_mesh_use_low_res"        value="${properties_cfg.get('front_top_lidar3d_c_mesh_use_low_res', True)}"/>
-  <xacro:property name="front_top_lidar3d_mount"                     value="2.0 0.0 2.0 0 ${0.5 * pi} 0"/>
-  <xacro:property name="use_left_top_lidar3d"                        value="${properties_cfg.get('use_left_top_lidar3d', True)}"/>
-  <xacro:property name="left_top_lidar3d_use_visual"                 value="${properties_cfg.get('left_top_lidar3d_use_visual', True)}"/>
-  <xacro:property name="left_top_lidar3d_use_collision"              value="${properties_cfg.get('left_top_lidar3d_use_collision', True)}"/>
-  <xacro:property name="left_top_lidar3d_color"                      value="0.0 0.0 0.0 1.0"/>
-  <xacro:property name="left_top_lidar3d_mount"                      value="0.10 0.6 1.35 0 0 ${0.5 * pi}"/>
-  <xacro:property name="use_chassis_imu"                             value="${properties_cfg.get('use_chassis_imu', True)}"/>
-  <xacro:property name="chassis_imu_mount"                           value="0.0 0.0 0.0 0.0 0.0 0.0"/>
-  <xacro:property name="use_fork_board_camera"                       value="${properties_cfg.get('use_fork_board_camera', True)}"/>
-  <xacro:property name="fork_board_camera_use_visual"                value="${properties_cfg.get('fork_board_camera_use_visual', True)}"/>
-  <xacro:property name="fork_board_camera_use_collision"             value="${properties_cfg.get('fork_board_camera_use_collision', True)}"/>
-  <xacro:property name="fork_board_camera_use_v_mesh"                value="${properties_cfg.get('fork_board_camera_use_v_mesh', True)}"/>
-  <xacro:property name="fork_board_camera_v_mesh_use_low_res"        value="${properties_cfg.get('fork_board_camera_v_mesh_use_low_res', True)}"/>
-  <xacro:property name="fork_board_camera_color"                     value="0.1 0.1 0.1 1.0"/>
-  <xacro:property name="fork_board_camera_use_c_mesh"                value="${properties_cfg.get('fork_board_camera_use_c_mesh', False)}"/>
-  <xacro:property name="fork_board_camera_c_mesh_use_low_res"        value="${properties_cfg.get('fork_board_camera_c_mesh_use_low_res', True)}"/>
-  <xacro:property name="fork_board_camera_mount"                     value="0.2 0.095 0.038 0 0 0"/>
+  <!--
+  ARGS
+  -->
+  <xacro:arg name="use_front_lidar2d"                    default="True"/>
+  <xacro:arg name="front_lidar2d_use_visual"             default="True"/>
+  <xacro:arg name="front_lidar2d_use_v_mesh"             default="True"/>
+  <xacro:arg name="front_lidar2d_v_mesh_use_low_res"     default="True"/>
+  <xacro:arg name="front_lidar2d_use_collision"          default="True"/>
+  <xacro:arg name="front_lidar2d_use_c_mesh"             default="False"/>
+  <xacro:arg name="front_lidar2d_c_mesh_use_low_res"     default="True"/>
+  <xacro:arg name="use_back_lidar2d"                     default="True"/>
+  <xacro:arg name="back_lidar2d_use_visual"              default="True"/>
+  <xacro:arg name="back_lidar2d_use_v_mesh"              default="True"/>
+  <xacro:arg name="back_lidar2d_v_mesh_use_low_res"      default="True"/>
+  <xacro:arg name="back_lidar2d_use_collision"           default="True"/>
+  <xacro:arg name="back_lidar2d_use_c_mesh"              default="False"/>
+  <xacro:arg name="back_lidar2d_c_mesh_use_low_res"      default="True"/>
+  <xacro:arg name="use_left_lidar2d"                     default="True"/>
+  <xacro:arg name="left_lidar2d_use_visual"              default="True"/>
+  <xacro:arg name="left_lidar2d_use_v_mesh"              default="True"/>
+  <xacro:arg name="left_lidar2d_v_mesh_use_low_res"      default="True"/>
+  <xacro:arg name="left_lidar2d_use_collision"           default="True"/>
+  <xacro:arg name="left_lidar2d_use_c_mesh"              default="False"/>
+  <xacro:arg name="left_lidar2d_c_mesh_use_low_res"      default="True"/>
+  <xacro:arg name="use_right_lidar2d"                    default="True"/>
+  <xacro:arg name="right_lidar2d_use_visual"             default="True"/>
+  <xacro:arg name="right_lidar2d_use_v_mesh"             default="True"/>
+  <xacro:arg name="right_lidar2d_v_mesh_use_low_res"     default="True"/>
+  <xacro:arg name="right_lidar2d_use_collision"          default="True"/>
+  <xacro:arg name="right_lidar2d_use_c_mesh"             default="False"/>
+  <xacro:arg name="right_lidar2d_c_mesh_use_low_res"     default="True"/>
+  <xacro:arg name="use_front_top_lidar3d"                default="True"/>
+  <xacro:arg name="front_top_lidar3d_use_visual"         default="True"/>
+  <xacro:arg name="front_top_lidar3d_use_v_mesh"         default="True"/>
+  <xacro:arg name="front_top_lidar3d_v_mesh_use_low_res" default="True"/>
+  <xacro:arg name="front_top_lidar3d_use_collision"      default="True"/>
+  <xacro:arg name="front_top_lidar3d_use_c_mesh"         default="False"/>
+  <xacro:arg name="front_top_lidar3d_c_mesh_use_low_res" default="True"/>
+  <xacro:arg name="use_left_top_lidar3d"                 default="True"/>
+  <xacro:arg name="left_top_lidar3d_use_visual"          default="True"/>
+  <xacro:arg name="left_top_lidar3d_use_collision"       default="True"/>
+  <xacro:arg name="use_fork_board_camera"                default="True"/>
+  <xacro:arg name="fork_board_camera_use_visual"         default="True"/>
+  <xacro:arg name="fork_board_camera_use_v_mesh"         default="True"/>
+  <xacro:arg name="fork_board_camera_v_mesh_use_low_res" default="True"/>
+  <xacro:arg name="fork_board_camera_use_collision"      default="True"/>
+  <xacro:arg name="fork_board_camera_use_c_mesh"         default="False"/>
+  <xacro:arg name="fork_board_camera_c_mesh_use_low_res" default="True"/>
+  <xacro:arg name="use_chassis_imu"                      default="True"/>
+  <!--
+  PROPERTIES
+  -->
+  <xacro:property name="use_front_lidar2d"                     value="$(arg use_front_lidar2d)"/>
+  <xacro:property name="front_lidar2d_use_visual"              value="$(arg front_lidar2d_use_visual)"/>
+  <xacro:property name="front_lidar2d_use_v_mesh"              value="$(arg front_lidar2d_use_v_mesh)"/>
+  <xacro:property name="front_lidar2d_v_mesh_use_low_res"      value="$(arg front_lidar2d_v_mesh_use_low_res)"/>
+  <xacro:property name="front_lidar2d_color"                   value="1 0.831372549 0.164705882 1"/>
+  <xacro:property name="front_lidar2d_use_collision"           value="$(arg front_lidar2d_use_collision)"/>
+  <xacro:property name="front_lidar2d_use_c_mesh"              value="$(arg front_lidar2d_use_c_mesh)"/>
+  <xacro:property name="front_lidar2d_c_mesh_use_low_res"      value="$(arg front_lidar2d_c_mesh_use_low_res)"/>
+  <xacro:property name="front_lidar2d_mount"                   value="2.1 0.0 -0.1 0 0 0"/>
+  <xacro:property name="use_back_lidar2d"                      value="$(arg use_back_lidar2d)"/>
+  <xacro:property name="back_lidar2d_use_visual"               value="$(arg back_lidar2d_use_visual)"/>
+  <xacro:property name="back_lidar2d_use_v_mesh"               value="$(arg back_lidar2d_use_v_mesh)"/>
+  <xacro:property name="back_lidar2d_v_mesh_use_low_res"       value="$(arg back_lidar2d_v_mesh_use_low_res)"/>
+  <xacro:property name="back_lidar2d_color"                    value="1 0.831372549 0.164705882 1"/>
+  <xacro:property name="back_lidar2d_use_collision"            value="$(arg back_lidar2d_use_collision)"/>
+  <xacro:property name="back_lidar2d_use_c_mesh"               value="$(arg back_lidar2d_use_c_mesh)"/>
+  <xacro:property name="back_lidar2d_c_mesh_use_low_res"       value="$(arg back_lidar2d_c_mesh_use_low_res)"/>
+  <xacro:property name="back_lidar2d_mount"                    value="-0.7 0.0 -0.1 0 0 ${-pi}"/>
+  <xacro:property name="use_left_lidar2d"                      value="$(arg use_left_lidar2d)"/>
+  <xacro:property name="left_lidar2d_use_visual"               value="$(arg left_lidar2d_use_visual)"/>
+  <xacro:property name="left_lidar2d_use_v_mesh"               value="$(arg left_lidar2d_use_v_mesh)"/>
+  <xacro:property name="left_lidar2d_v_mesh_use_low_res"       value="$(arg left_lidar2d_v_mesh_use_low_res)"/>
+  <xacro:property name="left_lidar2d_color"                    value="1 0.831372549 0.164705882 1"/>
+  <xacro:property name="left_lidar2d_use_collision"            value="$(arg left_lidar2d_use_collision)"/>
+  <xacro:property name="left_lidar2d_use_c_mesh"               value="$(arg left_lidar2d_use_c_mesh)"/>
+  <xacro:property name="left_lidar2d_c_mesh_use_low_res"       value="$(arg left_lidar2d_c_mesh_use_low_res)"/>
+  <xacro:property name="left_lidar2d_mount"                    value="0.4 0.7 -0.1 0 0 ${0.5 * pi}"/>
+  <xacro:property name="use_right_lidar2d"                     value="$(arg use_right_lidar2d)"/>
+  <xacro:property name="right_lidar2d_use_visual"              value="$(arg right_lidar2d_use_visual)"/>
+  <xacro:property name="right_lidar2d_use_v_mesh"              value="$(arg right_lidar2d_use_v_mesh)"/>
+  <xacro:property name="right_lidar2d_v_mesh_use_low_res"      value="$(arg right_lidar2d_v_mesh_use_low_res)"/>
+  <xacro:property name="right_lidar2d_color"                   value="1 0.831372549 0.164705882 1"/>
+  <xacro:property name="right_lidar2d_use_collision"           value="$(arg right_lidar2d_use_collision)"/>
+  <xacro:property name="right_lidar2d_use_c_mesh"              value="$(arg right_lidar2d_use_c_mesh)"/>
+  <xacro:property name="right_lidar2d_c_mesh_use_low_res"      value="$(arg right_lidar2d_c_mesh_use_low_res)"/>
+  <xacro:property name="right_lidar2d_mount"                   value="1.4 -0.7 -0.1 0 0 ${-0.5 * pi}"/>
+  <xacro:property name="use_front_top_lidar3d"                 value="$(arg use_front_top_lidar3d)"/>
+  <xacro:property name="front_top_lidar3d_use_visual"          value="$(arg front_top_lidar3d_use_visual)"/>
+  <xacro:property name="front_top_lidar3d_use_v_mesh"          value="$(arg front_top_lidar3d_use_v_mesh)"/>
+  <xacro:property name="front_top_lidar3d_v_mesh_use_low_res"  value="$(arg front_top_lidar3d_v_mesh_use_low_res)"/>
+  <xacro:property name="front_top_lidar3d_color"               value="0 0 0 1"/>
+  <xacro:property name="front_top_lidar3d_use_collision"       value="$(arg front_top_lidar3d_use_collision)"/>
+  <xacro:property name="front_top_lidar3d_use_c_mesh"          value="$(arg front_top_lidar3d_use_c_mesh)"/>
+  <xacro:property name="front_top_lidar3d_c_mesh_use_low_res"  value="$(arg front_top_lidar3d_c_mesh_use_low_res)"/>
+  <xacro:property name="front_top_lidar3d_mount"               value="2.0 0.0 2.0 0 ${0.5 * pi} 0"/>
+  <xacro:property name="use_left_top_lidar3d"                  value="$(arg use_left_top_lidar3d)"/>
+  <xacro:property name="left_top_lidar3d_use_visual"           value="$(arg left_top_lidar3d_use_visual)"/>
+  <xacro:property name="left_top_lidar3d_color"                value="0.0 0.0 0.0 1.0"/>
+  <xacro:property name="left_top_lidar3d_use_collision"        value="$(arg left_top_lidar3d_use_collision)"/>
+  <xacro:property name="left_top_lidar3d_mount"                value="0.10 0.6 1.35 0 0 ${0.5 * pi}"/>
+  <xacro:property name="use_chassis_imu"                       value="$(arg use_chassis_imu)"/>
+  <xacro:property name="chassis_imu_mount"                     value="0.0 0.0 0.0 0.0 0.0 0.0"/>
+  <xacro:property name="use_fork_board_camera"                 value="$(arg use_fork_board_camera)"/>
+  <xacro:property name="fork_board_camera_use_visual"          value="$(arg fork_board_camera_use_visual)"/>
+  <xacro:property name="fork_board_camera_use_v_mesh"          value="$(arg fork_board_camera_use_v_mesh)"/>
+  <xacro:property name="fork_board_camera_v_mesh_use_low_res"  value="$(arg fork_board_camera_v_mesh_use_low_res)"/>
+  <xacro:property name="fork_board_camera_color"               value="0.1 0.1 0.1 1.0"/>
+  <xacro:property name="fork_board_camera_use_collision"       value="$(arg fork_board_camera_use_collision)"/>
+  <xacro:property name="fork_board_camera_use_c_mesh"          value="$(arg fork_board_camera_use_c_mesh)"/>
+  <xacro:property name="fork_board_camera_c_mesh_use_low_res"  value="$(arg fork_board_camera_c_mesh_use_low_res)"/>
+  <xacro:property name="fork_board_camera_mount"               value="0.2 0.095 0.038 0 0 0"/>
   <!--
   ##############################################################################
